File: ThreePhase/Design/SAMS-LVMD/INV.kicad_sch (KiCad schematic)
At the start: 59 parts, among them J3 MOTOR OUTPUT, U1 U CHANNEL DRIVER, U2 V CHANNEL DRIVER, U3 W CHANNEL DRIVER, U4 ISEN 50mV/V, U5 ISEN 50mV/V, U6 ISEN 50mV/V

Commit message: 3P schematic update 6
Connections:
- net UEN renamed UINH
- net VEN renamed VINH
- net WEN renamed WINH
Changed lines of the file:
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@@
 		)
 	)
-	(hierarchical_label "WEN"
+	(hierarchical_label "WINH"
 		(shape input)
 		(at 30.48 139.7 180)
@@
 		)
 	)
-	(hierarchical_label "VEN"
+	(hierarchical_label "VINH"
 		(shape input)
 		(at 30.48 82.55 180)
@@
 		)
 	)
-	(hierarchical_label "UEN"
+	(hierarchical_label "UINH"
 		(shape input)
 		(at 30.48 25.4 180)

Commit message: 3P schematic update 7
Parts:
- removed R1, R2, R3, R4: 10K, SAMPI:RES0603, symbol SAMPI:RES
- removed R10, R5, R6, R7, R8, R9: 1K, SAMPI:RES0603, symbol SAMPI:RES
- D17, D18, D19: value 5V -> VZ3.3; MFT Toshiba -> Comchip Technology; MNP DF2S6.2FS,L3M -> CPDQ3V3-HF
- R25, R29, R34: value 100K -> 150K
Connections:
- net UIN: now also U1.2 (IN)
- net UINH: now also U1.3 (INH)
- net VIN: now also U2.2 (IN)
- net VINH: now also U2.3 (INH)
- net WIN: now also U3.2 (IN)
- net WINH: now also U3.3 (INH)
