File: ThreePhase/Design/SAMS-LVMD/MCU.kicad_sch (KiCad schematic)
At the start: 0 parts

Commit message: 3P schematic update 6
Parts:
- added U8: dsPIC33AKxxxMC106, SAMPI:TQFP64_10x10_MCHP, symbol SAMPI:dsPIC33AKxxxMC106

Commit message: 3P schematic update 7
Parts:
- added D1, D2, D3, D4, D5, D6, D7: VZ3.3, SAMPI:SOD-923, symbol SAMPI:TVS
- added R42, R43, R44, R45, R46, R47, R48: 10R, SAMPI:RES0603, symbol SAMPI:RES
Connections:
- net DIR_U: now also R42.2
- net DIR_V: now also R43.2
- net DIR_W: now also R44.2
- net FAULT: now also R48.2
- net PWM_U: now also R45.2
- net PWM_V: now also R46.2
- net PWM_W: now also R47.2
- new net: D5.1, R46.1
- new net: D3.1, R44.1
- new net: D7.1, R48.1
- new net: D1.1, R42.1
- new net: D2.1, R43.1
- new net: D4.1, R45.1
- new net: D6.1, R47.1
- new net GND: D1.2, D2.2, D3.2, D4.2, D5.2, D6.2, D7.2
