File: ThreePhase/Design/SAMS-LVMD/SAMS-LVMD.kicad_sch (KiCad schematic)
At the start: 49 parts, among them U1 U CHANNEL DRIVER, U2 V CHANNEL DRIVER, U3 W CHANNEL DRIVER, U4 ISEN 50mV/V, U5 ISEN 50mV/V, U6 ISEN 50mV/V

Commit message: 3P schematic update 1
Parts:
- C1, C11, C2, C3, C5, C8: footprint (none) -> SAMPI:CAP0603; MFT (none) -> Samsung; MNP (none) -> CL10A105KL8NNNC
- C10, C12, C13, C4, C6, C7, C9: footprint (none) -> SAMPI:CAP0603; MFT (none) -> Samsung; MNP (none) -> CL10C102JB8NNNC
- R1, R12, R8: footprint (none) -> SAMPI:RES0603; MFT (none) -> Yageo; MNP (none) -> RC0603JR-070RL
- R10, R15, R19: value SHUNT -> 10mR; footprint (none) -> SAMPI:SHUNT_1206; MFT (none) -> Yageo; MNP (none) -> RC0603JR-0710RL
- R11, R13, R16, R17, R20, R21: footprint (none) -> SAMPI:RES0603; MFT (none) -> Yageo; MNP (none) -> PE1206FKF470R01Z
- R14, R18, R22, R3, R4, R5, R6, R7, R9: footprint (none) -> SAMPI:RES0603; MFT (none) -> Yageo; MNP (none) -> RC0603JR-071KL
- R2, R24: footprint (none) -> SAMPI:RES0603; MFT (none) -> Yageo; MNP (none) -> RC0603JR-0710KL
- R23: footprint (none) -> SAMPI:RES0603; MFT (none) -> Yageo; MNP (none) -> RC0603JR-13100KL
- U1, U2, U3: MFT Infineon Technologies -> Infineon
- U4, U5, U6: Checked OK -> (none); Unit Price 0.079 -> (none)

Commit message: 3P schematic update 3
Parts:
- added C14, C15, C17: 1nF, SAMPI:CAP0603, symbol SAMPI:CERCAP
- added C16, C19: 1uF, SAMPI:CAP0603, symbol SAMPI:CERCAP
- added C18, C20, C21: 470uF/35V, symbol SAMPI:ELECCAP
- added D10, D11, D12, D13, D14, D15, D16, D7, D8: 5V, Liem:SOD-323_12, symbol SAMPI:TVS
- added D9: 24V, symbol Liem:DIODE-ZEN
- added J1: SIGNALS, symbol SAMPI:DIL14
- added J2: POWER INPUT, symbol Liem:SIL02
- added J3: MOTOR OUTPUT, symbol SAMPI:SIL03
- added Q1: 55V/42A, symbol Liem:FET_P-CH
- added R25, R26, R27, R30, R31, R32: 10K, SAMPI:RES0603, symbol SAMPI:RES
- added R28: 1K, SAMPI:RES0603, symbol SAMPI:RES
- added R29: 0R, SAMPI:RES0603, symbol SAMPI:RES
Connections:
- net +3V3: now also D16.1, J1.2
- net FAULT: now also D12.1, J1.9
- net GND: now also C14.1, C15.1, C16.1, C17.1, C18.-, C19.1, C20.-, C21.-, D10.2, D11.2, D12.2, D13.2, D14.2, D15.2, D16.2, D8.2, J1.1, J2.2, R25.1, R26.1, R27.1, R28.2, R29.2, R30.1, R31.1, R32.1; no longer C11.1, C12.1, C13.1, C5.1, C6.1, C8.1, C9.1, R24.1, U4.1 (REF), U4.2 (GND), U5.1 (REF), U5.2 (GND), U6.1 (REF), U6.2 (GND)
- net IU_SEN: now also J1.11
- net IV_SEN: now also J1.12
- net IW_SEN: now also J1.13
- net PHASE_U: now also C15.2, J3.1, R27.2
- net PHASE_V: now also C14.2, J3.2, R26.2
- net PHASE_W: now also C17.2, J3.3, R25.2
- net UEN: now also D8.1, J1.3, R30.2
- net UIN: now also D15.1, J1.4
- net VDC: now also C18.+, C19.2, C20.+, C21.+, D9.K, Q1.2 (S)
- net VDC_DIV: now also D7.1, J1.10
- net VEN: now also D10.1, J1.5, R31.2
- net VIN: now also D14.1, J1.6
- net WEN: now also D11.1, J1.7, R32.2
- net WIN: now also D13.1, J1.8
- new net: C16.2, J2.1, Q1.3 (D)
- new net: D9.A, Q1.1 (G), R28.1
- new net AGND: C11.1, C12.1, C13.1, C5.1, C6.1, C8.1, C9.1, D7.2, J1.14, R24.1, R29.1, U4.1 (REF), U4.2 (GND), U5.1 (REF), U5.2 (GND), U6.1 (REF), U6.2 (GND)
Other:
- moved on the sheet: C1, C10, C11, C12, C13, C2, C3, C4, C5, C6, C7, C8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

Commit message: 3P schematic update 4
Parts:
- C18, C20, C21: footprint (none) -> SAMPI:CAP_ELEC-10.3x10.3-DIA10
- D10, D11, D12, D13, D14, D15, D16, D7, D8: footprint Liem:SOD-323_12 -> SAMPI:SOD-923
- D9: footprint (none) -> SAMPI:SOD-123
- J1: footprint (none) -> SAMPI:IDC-2x7x2MM-TH
- Q1: footprint (none) -> SAMPI:D2PAK_TO-263
Changed lines of the file:
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@@
 			)
 		)
-		(property "Footprint" "Liem:SOD-323_12"
+		(property "Footprint" "SAMPI:SOD-923"
 			(at 274.955 69.85 0)
 			(effects
@@
 			)
 		)
-		(property "Footprint" "Liem:SOD-323_12"
+		(property "Footprint" "SAMPI:SOD-923"
 			(at 205.105 72.39 0)
 			(effects
@@
 			)
 		)
-		(property "Footprint" "Liem:SOD-323_12"
+		(property "Footprint" "SAMPI:SOD-923"
 			(at 217.805 72.39 0)
 			(effects
@@
 			)
 		)
-		(property "Footprint" "Liem:SOD-323_12"
+		(property "Footprint" "SAMPI:SOD-923"
 			(at 211.455 72.39 0)
 			(effects
@@
 			)
 		)
-		(property "Footprint" "Liem:SOD-323_12"
+		(property "Footprint" "SAMPI:SOD-923"
 			(at 198.755 72.39 0)
 			(effects
@@
 			)
 		)
-		(property "Footprint" ""
+		(property "Footprint" "SAMPI:CAP_ELEC-10.3x10.3-DIA10"
 			(at 204.47 101.6 0)
 			(effects
@@
 			)
 		)
-		(property "Footprint" ""
+		(property "Footprint" "SAMPI:SOD-123"
 			(at 254 106.68 0)
 			(effects
@@
 			)
 		)
-		(property "Footprint" "Liem:SOD-323_12"
+		(property "Footprint" "SAMPI:SOD-923"
 			(at 201.295 157.48 0)
 			(effects
@@
 			)
 		)
-		(property "Footprint" ""
+		(property "Footprint" "SAMPI:IDC-2x7x2MM-TH"
 			(at 231.14 50.8 0)
 			(effects
@@
 			)
 		)
-		(property "Footprint" ""
+		(property "Footprint" "SAMPI:CAP_ELEC-10.3x10.3-DIA10"
 			(at 217.17 101.6 0)
 			(effects
@@
 			)
 		)
-		(property "Footprint" ""
+		(property "Footprint" "SAMPI:CAP_ELEC-10.3x10.3-DIA10"
 			(at 229.87 101.6 0)
 			(effects
@@
 			)
 		)
-		(property "Footprint" "Liem:SOD-323_12"
+		(property "Footprint" "SAMPI:SOD-923"
 			(at 268.605 69.85 0)
 			(effects
@@
 			)
 		)
-		(property "Footprint" "Liem:SOD-323_12"
+		(property "Footprint" "SAMPI:SOD-923"
 			(at 255.905 69.85 0)
 			(effects
@@
 			)
 		)
-		(property "Footprint" ""
+		(property "Footprint" "SAMPI:D2PAK_TO-263"
 			(at 261.62 101.6 0)
 			(effects
@@
 			)
 		)
-		(property "Footprint" "Liem:SOD-323_12"
+		(property "Footprint" "SAMPI:SOD-923"
 			(at 262.255 69.85 0)
 			(effects

Commit message: 3P schematic update 5
Parts:
- removed C1, C11, C16, C19, C2, C3, C5, C8: 1uF, SAMPI:CAP0603, symbol SAMPI:CERCAP
- removed C10, C12, C13, C14, C15, C17, C4, C6, C7, C9: 1nF, SAMPI:CAP0603, symbol SAMPI:CERCAP
- removed C18, C20, C21: 470uF/35V, SAMPI:CAP_ELEC-10.3x10.3-DIA10, symbol SAMPI:ELECCAP
- removed D1, D2, D3, D4, D5, D6: 3A/40V, SAMPI:DO-214AB, symbol SAMPI:DIODE-SCH
- removed D12, D8: 5V, SAMPI:SOD-923, symbol SAMPI:TVS
- removed D9: 24V, SAMPI:SOD-123, symbol Liem:DIODE-ZEN
- removed J2: POWER INPUT, symbol Liem:SIL02
- removed J3: MOTOR OUTPUT, symbol SAMPI:SIL03
- removed Q1: 55V/42A, SAMPI:D2PAK_TO-263, symbol Liem:FET_P-CH
- removed R1, R12, R29, R8: 0R, SAMPI:RES0603, symbol SAMPI:RES
- removed R10, R15, R19: 10mR, SAMPI:SHUNT_1206, symbol SAMPI:SHUNT
- removed R11, R13, R16, R17, R20, R21: 10R, SAMPI:RES0603, symbol SAMPI:RES
- removed R14, R18, R22, R28, R3, R4, R5, R6, R7, R9: 1K, SAMPI:RES0603, symbol SAMPI:RES
- removed R2, R24, R25, R26, R27, R30, R31, R32: 10K, SAMPI:RES0603, symbol SAMPI:RES
- removed R23: 100K, SAMPI:RES0603, symbol SAMPI:RES
- removed U1: U CHANNEL DRIVER, SAMPI:TO-263-7, symbol SAMPI:BTS7960
- removed U2: V CHANNEL DRIVER, SAMPI:TO-263-7, symbol SAMPI:BTS7960
- removed U3: W CHANNEL DRIVER, SAMPI:TO-263-7, symbol SAMPI:BTS7960
- removed U4, U5, U6: ISEN 50mV/V, SAMPI:SOT363, symbol SAMPI:ZXCT199Q_INV
- added D9: 5V, SAMPI:SOD-923, symbol SAMPI:TVS
Connections:
- net +3V3: now also D7.1; no longer D16.1
- net AGND: no longer D7.2
- net FAULT: now also D16.1
- net GND: now also D7.2, D9.2
- net UEN: now also D13.1
- net UIN: now also D9.1; no longer D15.1
- net VDC_DIV: no longer D7.1
- net VEN: now also D14.1; no longer D10.1
- net VIN: now also D10.1; no longer D14.1
- net WEN: now also D15.1; no longer D11.1
- net WIN: now also D11.1; no longer D13.1
Other:
- added sheet INV (INV.kicad_sch)
- added sheet MCU (MCU.kicad_sch)
- added sheet PSU (PSU.kicad_sch)

Commit message: 3P schematic update 6
Other:
- added sheet DBG (DBG.kicad_sch)
- sheet INV ports: added UINH, VINH, WINH; removed UEN, VEN, WEN
- sheet PSU ports: added INV_EN; removed none
Changed lines of the file:
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@@
+	)
+	(sheet
+		(at 101.6 19.05)
+		(size 25.4 12.7)
+		(fields_autoplaced yes)
+		(stroke
+			(width 0.1524)
+			(type solid)
+		)
+		(fill
+			(color 255 254 201 1.0000)
+		)
+		(property "Sheetname" "DBG"
+			(at 101.6 18.3384 0)
+			(effects
+				(font
+					(size 1.27 1.27)
+				)
+				(justify left bottom)
+			)
+		)
+		(property "Sheetfile" "DBG.kicad_sch"
+			(at 101.6 32.3346 0)
+			(effects
+				(font
+					(size 1.27 1.27)
+				)
+				(justify left top)
+			)
+		)
+		(instances
+			(project "SAMS-LVMD"
+				(path "/eabd06f1-940c-48a8-9672-5070803c1e31"
+					(page "5")
+				)
+			)
+		)
 	)
 	(sheet
@@
 			)
 		)
+		(pin "INV_EN" input
+			(at 57.15 43.18 0)
+			(effects
+				(font
+					(size 1.27 1.27)
+				)
+				(justify right)
+			)
+		)
 		(instances
 			(project "SAMS-LVMD"
@@
 			)
 		)
-		(pin "WEN" input
+		(pin "WINH" input
 			(at 127 50.8 0)
 			(effects
@@
 			)
 		)
-		(pin "VEN" input
+		(pin "VINH" input
 			(at 127 46.355 0)
 			(effects
@@
 			)
 		)
-		(pin "UEN" input
+		(pin "UINH" input
 			(at 127 57.785 0)
 			(effects

Commit message: 3P schematic update 7
Parts:
- removed D10, D11, D13, D14, D15, D16, D7, D9: 5V, SAMPI:SOD-923, symbol SAMPI:TVS
- removed J1: SIGNALS, SAMPI:IDC-2x7x2MM-TH, symbol SAMPI:DIL14
Other:
- sheet PSU ports: added IDC_SEN; removed none
